File: pcb/keyboard.sch (KiCad schematic (older format))
At the start: 105 parts, among them J1 EXT-OLED, J2 AudioJack4, SW1 0, 0, SW10 1, 3, SW101 RST, SW102 BATT_EN, SW11 1, 4, SW12 1, 5, SW13 2, 0, SW14 2, 1, SW15 2, 2, SW16 2, 3, SW17 2, 4, SW18 2, 5, SW19 3, 0, SW2 0, 1, SW20 3, 1, SW21 3, 2, SW22 3, 3, SW23 3, 4, SW24 3, 5, SW25 4, 3, SW26 4, 4, SW27 4, 5, SW3 0, 2, SW4 0, 3, SW5 0, 4, SW6 0, 5, SW7 1, 0, SW8 1, 1, SW9 1, 2, U1 ProMicro

Commit message: pcb: cleanup & added schematics.pdf
Parts:
- LED1, LED10, LED11, LED12, LED13, LED14, LED15, LED16, LED17, LED18, LED19, LED2, LED20, LED21, LED22, LED23, LED24, LED25, LED26, LED27, LED3, LED4, LED5, LED6, LED7, LED8, LED9: symbol cornel-rescue:SK6812MINI-E-local -> cornel-rescue:SK6812MINI-E-local-cornel-rescue
Connections:
- net VCC is gone; now on net GND: J1.2 (Pin_2), J2.T, LED1.1 (VDD), LED10.1 (VDD), LED11.1 (VDD), LED12.1 (VDD), LED13.1 (VDD), LED14.1 (VDD), LED15.1 (VDD), LED16.1 (VDD), LED17.1 (VDD), LED18.1 (VDD), LED19.1 (VDD), LED2.1 (VDD), LED20.1 (VDD), LED21.1 (VDD), LED22.1 (VDD), LED23.1 (VDD), LED24.1 (VDD), LED25.1 (VDD), LED26.1 (VDD), LED27.1 (VDD), LED3.1 (VDD), LED4.1 (VDD), LED5.1 (VDD), LED6.1 (VDD), LED7.1 (VDD), LED8.1 (VDD), LED9.1 (VDD), R1.2, R2.2, U1.21 (VCC)
Other:
- note added: "*FIXME*\nreversing LED order might\nbe better than jumpers"
- note added: "BATTERY"
- note added: "PERIPHERALS"
- note added: "PWR CONN"
- moved on the sheet: BT1, C1, D1, D10, D101, D11, D12, D13, D14, D15, D16, D17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
